File: Hardware/Schematic 1.0.sch (EAGLE design)
At the start: 2 parts, among them U2 ATMEGA328P-AU

Commit message: Added Newest Hardware
Parts:
- added FTDI_HEADER: (no value), pinhead:PINHD-1X6
- added J1: AVR-ISP-6PINAVR-ISP-6PIN-SMALL-SILK, avr-isp:AVR-ISP-6PINAVR-ISP-6PIN-SMALL-SILK
- added JP1: (no value), pinhead:PINHD-2X12
Connections:
- new net 1/PD3/BLE_MOD: JP1.19, U2.PD3
- new net 10/PD6/BLE_RTS: JP1.22, U2.PD6
- new net 32/PD2/BLE_CTS: JP1.18, U2.PD2
- new net N$10: J1.2
- new net NS10: C1.1
- new net PB0: JP1.1, U2.PB0
- new net PC0: JP1.9, U2.PC0
- new net PC1: JP1.10, U2.PC1
- new net PC4: JP1.13, U2.PC4
- new net PC5: JP1.14, U2.PC5
- new net PD7: JP1.23, U2.PD7
- new net XTAL2: C1.2
- net 13/PB1/LCD_C/!D: now also JP1.2
- net 14/PB2/!LCD_CS: now also JP1.3
- net 15/PB3/MOSI: now also J1.4, JP1.4
- net 16/PB4/MISO: now also J1.1, JP1.5
- net 17/PB5/SCK: now also J1.3, JP1.6
- net 19/ADC6: now also JP1.24
- net 2/PD4/LCD_X+: now also JP1.20
- net 25/PC2/LCD_Y+: now also JP1.11
- net 26/PC3/LCD_X-: now also JP1.12
- net 29/PC6/!RESET: now also FTDI_HEADER.1, J1.5, JP1.15
- net 9/PD5/LCD_Y-: now also JP1.21
- net ATRXD_BLTXD: now also FTDI_HEADER.2, JP1.16
- net ATTXD_BLRXD: now also FTDI_HEADER.3, JP1.17
- net GND: now also C1.1, FTDI_HEADER.5, FTDI_HEADER.6, J1.6, JP1.8
- net VCC: now also FTDI_HEADER.4, JP1.7; no longer C1.1
Other:
- moved on the sheet: C1
